File: Kicad/Paikorea.kicad_pcb (KiCad board)
At the start: 2 copper layers, 137.9 x 78 mm, 54 parts, among them J1 AudioJack3, J2 TPS43-201A-S, J3 TPS43-201A-S, J4 AudioJack3, K10 PG1316S, K11 PG1316S, K12 PG1316S, K13 PG1316S, K14 PG1316S, K15 PG1316S, K16 PG1316S, K17 PG1316S, K18 PG1316S, K19 PG1316S, K20 PG1316S, K21 PG1316S, K22 PG1316S, K4 PG1316S, K5 PG1316S, K6 PG1316S, K7 PG1316S, K8 PG1316S, K9 PG1316S, U1 RP2040-Zero, U2 RP2040-Zero

Commit message: .
Parts:
- removed J3: TPS43-201A-S, DreaM117er-keebLibrary:Hirose_FH12-6S-0.5SH_1x06-1MP_P0.50mm_Horizontal
- removed N10, N11, N12, N9: MAC8 TH1.6-0.3 M2, DreaM117er-keebLibrary:MAC8_TH0816-XX-M2-Dual_Pad
Connections:
- J2 pad 1: SDA_B -> SDA
- J2 pad 2: SCL_B -> SCL
- U1 pad 16: unconnected-(U1-GP15-Pad16) -> SDA
- U1 pad 17: unconnected-(U1-GP26-Pad17) -> SCL
- U1 pad 7: SDA -> unconnected-(U1-GP6-Pad7)
- U1 pad 8: SCL -> unconnected-(U1-GP7-Pad8)
Routing:
- net +3V3: track 126.8 -> 49.8 mm, vias 1 -> 0
- net SDA_B: track 38.7 -> 0.00 mm, vias 1 -> 0
- net SCL_B: track 37.8 -> 0.00 mm, vias 1 -> 0
- net GND: track 79.0 -> 45.7 mm
- net SCL: track 18.8 -> 39.2 mm, vias 1 -> 0
- net row3: track 187.1 -> 171.6 mm
- net SDA: track 20.5 -> 36.0 mm, vias 1 -> 0
- net +5V: track 165.6 -> 162.3 mm
