File: Kicad/Paikorea.kicad_pcb (KiCad board)
At the start: 2 copper layers, 137.9 x 78 mm, 49 parts, among them J1 AudioJack3, J2 TPS43-201A-S, J4 AudioJack3, K10 PG1316S, K11 PG1316S, K12 PG1316S, K13 PG1316S, K14 PG1316S, K15 PG1316S, K16 PG1316S, K17 PG1316S, K18 PG1316S, K19 PG1316S, K20 PG1316S, K21 PG1316S, K22 PG1316S, K4 PG1316S, K5 PG1316S, K6 PG1316S, K7 PG1316S, K8 PG1316S, K9 PG1316S, U1 RP2040-Zero, U2 RP2040-Zero

Commit message: RP2040-Zero: use footprint/RP2040-Zero geometry, same GPIO numbers on front/back
- U1 (F) / U2 (B): new footprint Paikorea:RP2040-Zero_UpsideDown, derived from
  footprint/RP2040-Zero.kicad_mod (mirrored for upside-down mounting, holes removed -> SMD pads)
- Both modules now use the same GPIO numbers:
  GP0 col5, GP1 col4, GP2 col3, GP3 col2, GP4 col1, GP5 row0, GP6 row1, GP7 row2,
  GP8 SDA, GP9 SCL (I2C0), GP10 row3, GP11 Data
- Rerouted MCU area: left (F) fan-out crosses under the module and joins the right (B)
  fan-out through a via ladder; I2C/3V3/GND to J2, 5V/Data to TRRS
- Zone fills cleared (refill with B)

Co-Authored-By: Claude Opus 5.5 <noreply@anthropic.com>
Claude-Session: https://claude.ai/code/session_01CM6fo4n92yZJeCtkGbFXPU
Parts:
- U1, U2: footprint Paikorea:RP2040_Zero_UpsideDown -> Paikorea:RP2040-Zero_UpsideDown
Connections:
- U1 pad 1: unconnected-(U1-GP0-Pad1) -> col5
- U1 pad 10: row2 -> SCL
- U1 pad 11: row1 -> row3
- U1 pad 13: row0 -> unconnected-(U1-GP12-Pad13)
- U1 pad 14: col1 -> unconnected-(U1-GP13-Pad14)
- U1 pad 15: col2 -> unconnected-(U1-GP14-Pad15)
- U1 pad 16: SDA -> unconnected-(U1-GP15-Pad16)
- U1 pad 17: SCL -> unconnected-(U1-GP26-Pad17)
- U1 pad 18: col3 -> unconnected-(U1-GP27-Pad18)
- U1 pad 19: col4 -> unconnected-(U1-GP28-Pad19)
- U1 pad 2: unconnected-(U1-GP1-Pad2) -> col4
- U1 pad 20: col5 -> unconnected-(U1-GP29-Pad20)
- U1 pad 3: unconnected-(U1-GP2-Pad3) -> col3
- U1 pad 4: unconnected-(U1-GP3-Pad4) -> col2
- U1 pad 5: unconnected-(U1-GP4-Pad5) -> col1
- U1 pad 6: unconnected-(U1-GP5-Pad6) -> row0
- U1 pad 7: unconnected-(U1-GP6-Pad7) -> row1
- U1 pad 8: unconnected-(U1-GP7-Pad8) -> row2
- U1 pad 9: row3 -> SDA
- U2 pad 1: unconnected-(U2-GP0-Pad1) -> col5
- U2 pad 10: col1 -> SCL
- U2 pad 11: row0 -> row3
- U2 pad 13: row1 -> unconnected-(U2-GP12-Pad13)
- U2 pad 14: row2 -> unconnected-(U2-GP13-Pad14)
- U2 pad 15: row3 -> unconnected-(U2-GP14-Pad15)
- U2 pad 2: unconnected-(U2-GP1-Pad2) -> col4
- U2 pad 3: unconnected-(U2-GP2-Pad3) -> col3
- U2 pad 4: col5 -> col2
- U2 pad 5: col4 -> col1
- U2 pad 6: col3 -> row0
- U2 pad 7: SDA_B -> row1
- U2 pad 8: SCL_B -> row2
- U2 pad 9: col2 -> SDA
Routing:
- net col5: track 134.3 -> 206.3 mm
- net col4: track 130.9 -> 197.8 mm
- net col2: track 129.6 -> 193.9 mm
- net col3: track 147.5 -> 211.4 mm
- net +3V3: track 49.8 -> 107.5 mm, vias 0 -> 1
- net col1: track 169.8 -> 226.0 mm
- net row0: track 199.9 -> 247.0 mm
- net GND: track 45.7 -> 87.2 mm, vias 2 -> 1
- net row1: track 186.5 -> 221.3 mm, vias 8 -> 7
- net row2: track 178.0 -> 202.5 mm, vias 7 -> 6
- net SDA: track 36.0 -> 53.2 mm, vias 0 -> 2
- net row3: track 171.6 -> 175.0 mm, vias 6 -> 5
- net SCL: track 39.2 -> 42.1 mm, vias 0 -> 2
- net +5V: track 162.3 -> 164.4 mm
