File: Kicad/Paikorea.kicad_pcb (KiCad board)
At the start: 2 copper layers, 137.9 x 78 mm, 49 parts, among them J1 AudioJack3, J2 TPS43-201A-S, J4 AudioJack3, K10 PG1316S, K11 PG1316S, K12 PG1316S, K13 PG1316S, K14 PG1316S, K15 PG1316S, K16 PG1316S, K17 PG1316S, K18 PG1316S, K19 PG1316S, K20 PG1316S, K21 PG1316S, K22 PG1316S, K4 PG1316S, K5 PG1316S, K6 PG1316S, K7 PG1316S, K8 PG1316S, K9 PG1316S, U1 RP2040-Zero, U2 RP2040-Zero

Commit message: .
Connections:
- U2 pad 10: SCL -> unconnected-(U2-GP9-Pad10)
- U2 pad 9: SDA -> unconnected-(U2-GP8-Pad9)
Routing:
- net SDA: track 53.2 -> 48.1 mm
- net GND: track 87.2 -> 92.1 mm
- net +5V: track 164.4 -> 159.7 mm
- net SCL: track 42.1 -> 39.5 mm
- net col5: track 206.3 -> 204.7 mm
