File: Kicad/Paikorea.kicad_pcb (KiCad board)
At the start: 2 copper layers, 137.9 x 78 mm, 49 parts, among them J1 AudioJack3, J2 TPS43-201A-S, J4 AudioJack3, K10 PG1316S, K11 PG1316S, K12 PG1316S, K13 PG1316S, K14 PG1316S, K15 PG1316S, K16 PG1316S, K17 PG1316S, K18 PG1316S, K19 PG1316S, K20 PG1316S, K21 PG1316S, K22 PG1316S, K4 PG1316S, K5 PG1316S, K6 PG1316S, K7 PG1316S, K8 PG1316S, K9 PG1316S, U1 RP2040-Zero, U2 RP2040-Zero

Commit message: .
Parts:
- J1, J4: footprint Connector_Audio:Jack_3.5mm_KoreanHropartsElec_PJ-320D-4A_Horizontal -> Paikorea:AUDIO-SMD_PJ-320D-1
- U1, U2: footprint Paikorea:RP2040-Zero_UpsideDown -> Paikorea:RP2040-Zero-smd
- moved U1 16.3 mm to (172.6, 87.7)
- moved U2 16.3 mm to (192.9, 87.7)
- moved J1 1.30 mm to (172.1, 122.9)
- moved J4 1.30 mm to (172.1, 122.9)
Routing:
- net Data: track 69.4 -> 73.4 mm
- net +5V: track 159.7 -> 161.6 mm
